File: atari_mods.kicad_pcb (KiCad board)
At the start: 2 copper layers, 33 x 35.6 mm, 14 parts, among them IC1 78L05F, J1 AVR-ISP-6, J2 Conn_01x02_Male, J3 DIN13T, J4 Conn_01x15_Female, SW1 Elec K2-1823SA-A4DW-06, U1 ATtiny85-20SU, U2 AUDIO-JACK3, U3 TS5V330

Commit message: first commit
Parts:
- removed U2: AUDIO-JACK3, libs:Tayda_3.5mm_stereo_TRS_jack_A-853
- added J5: AudioJack3_Ground, kicad-footprints:Jack_3.5mm_Switronic_ST-005-G_horizontal, F.Cu at (108.0, 100.4)
- SW1, U3: moved to B.Cu
- moved SW1 41.4 mm to (136.6, 114.4)
- moved J2 18.8 mm to (132.8, 111.0), turned to 90 degrees
- moved J1 15.5 mm to (120.0, 100.7)
- moved U3 15.3 mm to (109.7, 111.9), turned to 180 degrees
- moved IC1 3.64 mm to (131.7, 115.3), turned to 0 degrees
- moved JP1 1.64 mm to (128.4, 110.3), turned to 90 degrees
- moved TM1 1.58 mm to (109.8, 107.2), turned to 180 degrees
- moved TM2 1.30 mm to (109.8, 111.5), turned to 180 degrees
- moved TM3 1.05 mm to (109.7, 115.7), turned to 180 degrees
- moved J3 0.76 mm to (120.7, 111.3)
- moved U1 0.58 mm to (131.7, 103.0)
- moved J4 0.44 mm to (125.2, 122.6)
Routing:
- net GND: track 25.5 -> 138.2 mm, vias 0 -> 4
- net +5V: track 0.00 -> 47.1 mm, vias 0 -> 3
- net /video_mod/H-SYNC: track 0.00 -> 40.6 mm, vias 0 -> 2
- net /video_mod/V-SYNC: track 0.00 -> 37.2 mm
- net /video_mod/AUDIOPOT: track 0.00 -> 30.6 mm
- net /video_mod/VRED: track 0.00 -> 25.9 mm, vias 0 -> 2
- net Net-(JP1-Pad2): track 0.00 -> 23.4 mm
- net /video_mod/MONOSIGNAL: track 0.00 -> 23.1 mm
- net /video_mod/AAUDIO: track 0.00 -> 20.3 mm, vias 0 -> 2
- net /video_mod/MISO: track 0.00 -> 18.7 mm, vias 0 -> 1
- net /video_mod/MOSI: track 0.00 -> 18.3 mm, vias 0 -> 1
- net /video_mod/VBLUE: track 0.00 -> 18.1 mm, vias 0 -> 1
- net /video_mod/VGREEN: track 0.00 -> 13.8 mm
- net /video_mod/SELECT: track 0.00 -> 12.5 mm
- net /video_mod/RST: track 0.00 -> 12.0 mm
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- added copper zone on B.Cu, net GND
- added copper zone on F.Cu, net GND
