File: video_mod.sch (KiCad schematic (older format))
At the start: 0 parts

Commit message: first commit
Parts:
- added IC1: 78L05F, kicad-footprints:SOT-89-3_Handsoldering, symbol mk6-eagle-import:78LF
- added J1: AVR-ISP-6, kicad-footprints:PinHeader_2x03_P1.27mm_Vertical, symbol Connector:AVR-ISP-6
- added J2: Conn_01x02_Male, kicad-footprints:PinHeader_1x02_P1.27mm_Vertical, symbol Connector:Conn_01x02_Male
- added J3: DIN13T, libs:ADADS, symbol Connector:Conn_01x13_Male
- added J4: Conn_01x15_Female, kicad-footprints:DSUB-15-HD_Female_Vertical_P2.29x1.98mm_MountingHoles, symbol Connector:Conn_01x15_Female
- added JP1: SolderJumper_3_Open, kicad-footprints:SolderJumper-3_P1.3mm_Open_Pad1.0x1.5mm, symbol Jumper:SolderJumper_3_Open
- added RV1: DB-1001N, libs:THUMB_POT, symbol Device:R_POT
- added SW1: Elec K2-1823SA-A4DW-06, libs:K2-1823SA, symbol Switch:SW_SPST
- added TM1, TM2, TM3: 100R, kicad-footprints:Potentiometer_Bourns_TC33X_Vertical, symbol mk6-eagle-import:TRIMPOTTC33X
- added U1: ATtiny85-20SU, kicad-footprints:SOIJ-8_5.3x5.3mm_P1.27mm, symbol MCU_Microchip_ATtiny:ATtiny85-20SU
- added U2: AUDIO-JACK3, libs:Tayda_3.5mm_stereo_TRS_jack_A-853, symbol mk6-eagle-import:AUDIO-JACK3
- added U3: TS5V330, kicad-footprints:SOIC-16_4.55x10.3mm_P1.27mm, symbol mk6-eagle-import:V330SO16L
Connections:
- new net: J2.1 (Pin_1), SW1.1 (A), U1.3 (XTAL2/PB4)
- new net: JP1.2 (C), U1.7 (PB2)
- new net: TM3.2 (S), U3.10 (S2C)
- new net: TM1.2 (S), U3.3 (S2A)
- new net: TM2.2 (S), U3.6 (S2B)
- new net +5V: IC1.1 (VO), J1.2 (VCC), U1.8 (VCC), U3.16 (VCC)
- new net AAUDIO: J3.1 (Pin_1), RV1.1
- new net ABLUE: J3.10 (Pin_10), TM3.1 (A)
- new net AGREEN: J3.6 (Pin_6), TM2.1 (A)
- new net ARED: J3.7 (Pin_7), TM1.1 (A)
- new net AUDIOPOT: RV1.2, U2.RING1, U2.TIP
- new net AVIDEO: J3.2 (Pin_2), U2.EARTH
- new net GND: IC1.2 (GND), IC1.2@1 (GND@1), J1.6 (GND), J2.2 (Pin_2), J3.13 (Pin_13), J4.10 (Pin_10), J4.5 (Pin_5), J4.6 (Pin_6), J4.7 (Pin_7), J4.8 (Pin_8), RV1.3, SW1.2 (B), TM1.3 (E), TM2.3 (E), TM3.3 (E), U1.4 (GND), U2.RING2, U3.12 (DD), U3.13 (S2D), U3.14 (S1D), U3.15 (EN), U3.8 (GND)
- new net H-SYNC: J3.9 (Pin_9), J4.13 (Pin_13), JP1.1 (A)
- new net MISO: J1.1 (MISO), U1.6 (PB1)
- new net MONOSIGNAL: J3.11 (Pin_11), U3.11 (S1C), U3.2 (S1A), U3.5 (S1B)
- new net MOSI: J1.4 (MOSI), U1.5 (AREF/PB0)
- new net RST: J1.5 (~RST), U1.1 (~RESET~/PB5)
- new net SCK: J1.3 (SCK), U1.2 (XTAL1/PB3)
- new net SELECT: J3.4 (Pin_4), U3.1 (IN)
- new net V-SYNC: J3.12 (Pin_12), J4.14 (Pin_14), JP1.3 (B)
- new net VBLUE: J4.3 (Pin_3), U3.9 (DC)
- new net VCC: IC1.3 (VI), J3.8 (Pin_8)
- new net VGREEN: J4.2 (Pin_2), U3.7 (DB)
- new net VRED: J4.1 (Pin_1), U3.4 (DA)
- no-connect marks 0 -> 7
Other:
- note added: "ATARI input"
- note added: "ATTINY procesor switcher"
- note added: "ATTINY programing interface"
- note added: "VGA output"
- note added: "multiplexer"
- note added: "power"
- note added: "sound"

Commit message: first commit
Parts:
- removed U2: AUDIO-JACK3, libs:Tayda_3.5mm_stereo_TRS_jack_A-853, symbol mk6-eagle-import:AUDIO-JACK3
- added J5: AudioJack3_Ground, kicad-footprints:Jack_3.5mm_Switronic_ST-005-G_horizontal, symbol Connector:AudioJack3_Ground
- IC1: symbol mk6-eagle-import:78LF -> atari_mods-rescue:78LF-mk6-eagle-import
- TM1, TM2, TM3: symbol mk6-eagle-import:TRIMPOTTC33X -> atari_mods-rescue:TRIMPOTTC33X-mk6-eagle-import
- U3: symbol mk6-eagle-import:V330SO16L -> atari_mods-rescue:V330SO16L-mk6-eagle-import
Connections:
- net AUDIOPOT: now also J5.R, J5.T
- net GND: now also J5.S
Changed lines of the file:
@@
 	2600 5450 2600 5600
 $Comp
-L mk6-eagle-import:AUDIO-JACK3 U2
-U 1 1 5F478DD6
-P 5850 5050
-F 0 "U2" H 5833 5452 59  0000 C CNN
-F 1 "AUDIO-JACK3" H 5900 5350 59  0000 C CNN
-F 2 "libs:Tayda_3.5mm_stereo_TRS_jack_A-853" H 5850 5050 50  0001 C CNN
-F 3 "" H 5850 5050 50  0001 C CNN
-	1    5850 5050
-	1    0    0    -1
-$EndComp
-$Comp
-L mk6-eagle-import:78LF IC?
+L atari_mods-rescue:78LF-mk6-eagle-import IC?
 U 1 1 5F47D0CF
 P 2700 1250
@@
 Text Label 6250 5050 0    50   ~ 0
 AUDIOPOT
-Wire Wire Line
-	6250 5050 6050 5050
-Wire Wire Line
-	6050 5050 6050 4950
-Wire Wire Line
-	6050 5050 6050 5150
-Connection ~ 6050 5050
-Wire Wire Line
-	6250 4850 6050 4850
-Text Label 6250 4850 0    50   ~ 0
-AVIDEO
 $Comp
 L power:GND #PWR010
 U 1 1 5F4B966F
-P 6250 5350
-F 0 "#PWR010" H 6250 5100 50  0001 C CNN
-F 1 "GND" H 6255 5177 50  0000 C CNN
-F 2 "" H 6250 5350 50  0001 C CNN
-F 3 "" H 6250 5350 50  0001 C CNN
-	1    6250 5350
-	1    0    0    -1
-$EndComp
-Wire Wire Line
-	6250 5350 6250 5250
-Wire Wire Line
-	6250 5250 6050 5250
+P 6150 5350
+F 0 "#PWR010" H 6150 5100 50  0001 C CNN
+F 1 "GND" H 6155 5177 50  0000 C CNN
+F 2 "" H 6150 5350 50  0001 C CNN
+F 3 "" H 6150 5350 50  0001 C CNN
+	1    6150 5350
+	1    0    0    -1
+$EndComp
 Wire Notes Line
 	6750 5950 6750 3350
@@
 sound
 $Comp
-L mk6-eagle-import:V330SO16L U3
+L atari_mods-rescue:V330SO16L-mk6-eagle-import U3
 U 1 1 5F4C3820
 P 7350 2200
@@
 $EndComp
 $Comp
-L mk6-eagle-import:TRIMPOTTC33X TM1
+L atari_mods-rescue:TRIMPOTTC33X-mk6-eagle-import TM1
 U 1 1 5F4C4ABC
 P 5450 1450
@@
 $EndComp
 $Comp
-L mk6-eagle-import:TRIMPOTTC33X TM2
+L atari_mods-rescue:TRIMPOTTC33X-mk6-eagle-import TM2
 U 1 1 5F4C6BAC
 P 5450 2050
@@
 $EndComp
 $Comp
-L mk6-eagle-import:TRIMPOTTC33X TM3
+L atari_mods-rescue:TRIMPOTTC33X-mk6-eagle-import TM3
 U 1 1 5F4C74CB
 P 8700 2200
@@
 Wire Wire Line
 	2600 6500 2600 6650
-Text Label 6050 5250 0    50   ~ 0
+Text Label 6150 5250 0    50   ~ 0
 GND
 Text Label 8150 2200 0    50   ~ 0
@@
 Wire Wire Line
 	3600 4650 3750 4650
+$Comp
+L Connector:AudioJack3_Ground J5
+U 1 1 5F49E77A
+P 5700 5050
+F 0 "J5" H 5682 5375 50  0000 C CNN
+F 1 "AudioJack3_Ground" H 5682 5284 50  0000 C CNN
+F 2 "kicad-footprints:Jack_3.5mm_Switronic_ST-005-G_horizontal" H 5700 5050 50  0001 C CNN
+F 3 "~" H 5700 5050 50  0001 C CNN
+	1    5700 5050
+	1    0    0    -1
+$EndComp
+Wire Wire Line
+	5900 5150 6000 5150
+Wire Wire Line
+	6000 5150 6000 5050
+Wire Wire Line
+	6000 5050 6250 5050
+Wire Wire Line
+	6000 5050 5900 5050
+Connection ~ 6000 5050
+Wire Wire Line
+	6150 4950 5900 4950
+Wire Wire Line
+	6150 4950 6150 5350
 $EndSCHEMATC
